Commit message: Improve visuals, and fix localisation and controller problems found by testing
Appearance
- world: PBR materials, three-light setup with shadows, dark skirting boards and
  bands at LiDAR height, plus a table, a third crate and a planter so scan
  matching has distinguishable features instead of identical flat walls
- robot: slate chassis with a blue deck, orange front bumper, a marked scan band
  on the LiDAR and a lens on the camera. All are extra visual elements on links
  that already existed, so collision, inertia and TF are unchanged
- two fixed camera sensors in the world for documentation images: Gazebo's GUI
  crashes on a virtual framebuffer, but its sensors render on the GPU headless

Localisation
- AMCL used 60 of 360 beams, too little to fix heading; a 2 degree heading error
  throws a 7 m return sideways by 24 cm. Raised to 180 beams, tightened the
  update thresholds and lowered the motion-noise alphas for simulated odometry.
  Measured with a new alignment check: returns landing exactly on a mapped wall
  cell went from 24% to 83%, returns falling outside the map from 15% to 0%,
  mean error from 7.9 cm to 0.9 cm
- the remaining half of that symptom was RViz parallax, not localisation: the
  map draws at z=0 and the returns at the LiDAR's 0.17 m, so a tilted camera
  offsets them. The RViz configs now default to a near-top-down view
- denser SLAM keyframes, 0.3 to 0.15 m and rad, for a sharper map

Control
- DWB kept stalling in tight spaces and reporting a lack of progress. Switched
  to Regulated Pure Pursuit and reduced the inflation radius to 0.45 m;
  recoveries went from 2 per goal to 0
- navigation.launch.py now lists the seven Nav2 nodes this project uses instead
  of including nav2_bringup. docking_server, which is unused here, once timed
  out sending its lifecycle response and left the whole navigation stack
  inactive, rejecting every goal with nothing logged as an error
- RViz gets Nav2's official tool set plus the Navigation 2 panel, so goal
  sending and stack status are visible rather than guessed at

Co-Authored-By: Claude Opus 5 <noreply@anthropic.com>

File: src/smartphone_robot/urdf/robot.urdf.xacro (robot description, xacro)
@@ -48,9 +48,13 @@
   <xacro:property name="PI" value="3.14159265359"/>
   <!-- ==================== Materials (RViz colours only) ================== -->
-  <material name="grey">   <color rgba="0.4 0.4 0.4 1.0"/></material>
-  <material name="black">  <color rgba="0.1 0.1 0.1 1.0"/></material>
-  <material name="blue">   <color rgba="0.2 0.3 0.8 1.0"/></material>
-  <material name="red">    <color rgba="0.8 0.2 0.2 1.0"/></material>
-  <material name="white">  <color rgba="0.9 0.9 0.9 1.0"/></material>
+  <material name="chassis">  <color rgba="0.26 0.29 0.36 1.0"/></material>
+  <material name="deck">     <color rgba="0.20 0.58 0.86 1.0"/></material>
+  <material name="tyre">     <color rgba="0.08 0.08 0.09 1.0"/></material>
+  <material name="hub">      <color rgba="0.62 0.64 0.68 1.0"/></material>
+  <material name="grey">     <color rgba="0.45 0.47 0.52 1.0"/></material>
+  <material name="sensor">   <color rgba="0.18 0.19 0.23 1.0"/></material>
+  <material name="lens">     <color rgba="0.10 0.35 0.55 1.0"/></material>
+  <material name="marker">   <color rgba="0.92 0.36 0.18 1.0"/></material>
+  <material name="white">    <color rgba="0.88 0.89 0.92 1.0"/></material>
   <!-- ==================== base_footprint =================================
        The tree's root: a massless frame on the GROUND directly below the robot's
@@ -71,10 +75,34 @@
   </joint>
   <link name="base_link">
-    <visual>
+    <!-- Several visual elements on one link. URDF allows this, and it costs nothing:
+         collision and inertia are unchanged, so physics and TF are identical. Only
+         what RViz and Gazebo draw is different. -->
+    <visual name="chassis">
       <origin xyz="0 0 ${base_height/2}" rpy="0 0 0"/>
       <geometry>
         <box size="${base_length} ${base_width} ${base_height}"/>
       </geometry>
-      <material name="blue"/>
+      <material name="chassis"/>
+    </visual>
+    <visual name="deck">
+      <origin xyz="-0.01 0 ${base_height + 0.008}" rpy="0 0 0"/>
+      <geometry>
+        <box size="${base_length*0.82} ${base_width*0.88} 0.016"/>
+      </geometry>
+      <material name="deck"/>
+    </visual>
+    <visual name="front_bumper">
+      <origin xyz="${base_length/2 - 0.012} 0 ${base_height*0.42}" rpy="0 0 0"/>
+      <geometry>
+        <box size="0.024 ${base_width*0.94} ${base_height*0.55}"/>
+      </geometry>
+      <material name="marker"/>
+    </visual>
+    <visual name="rear_panel">
+      <origin xyz="${-base_length/2 + 0.010} 0 ${base_height*0.5}" rpy="0 0 0"/>
+      <geometry>
+        <box size="0.020 ${base_width*0.80} ${base_height*0.6}"/>
+      </geometry>
+      <material name="grey"/>
     </visual>
     <collision>
@@ -107,9 +135,26 @@
     </joint>
     <link name="${prefix}_wheel_link">
-      <visual>
+      <visual name="tyre">
         <geometry>
           <cylinder radius="${wheel_radius}" length="${wheel_width}"/>
         </geometry>
-        <material name="black"/>
+        <material name="tyre"/>
+      </visual>
+      <!-- A hub that is visibly off-centre in rotation, so wheel spin is obvious in
+           RViz and in the Gazebo GUI. Useful when checking that the differential drive
+           plugin is actually turning the joints. -->
+      <visual name="hub">
+        <origin xyz="0 0 ${wheel_width/2 + 0.001}" rpy="0 0 0"/>
+        <geometry>
+          <cylinder radius="${wheel_radius*0.45}" length="0.004"/>
+        </geometry>
+        <material name="hub"/>
+      </visual>
+      <visual name="spoke">
+        <origin xyz="${wheel_radius*0.6} 0 ${wheel_width/2 + 0.002}" rpy="0 0 0"/>
+        <geometry>
+          <box size="${wheel_radius*0.55} 0.008 0.004"/>
+        </geometry>
+        <material name="marker"/>
       </visual>
       <collision>
@@ -160,9 +205,26 @@
   </joint>
   <link name="lidar_link">
-    <visual>
+    <visual name="lidar_body">
       <geometry>
         <cylinder radius="${lidar_radius}" length="${lidar_height}"/>
       </geometry>
-      <material name="red"/>
+      <material name="sensor"/>
+    </visual>
+    <!-- The orange band sits at the scan plane, which makes it easy to see at a glance
+         how high the LiDAR actually measures and what it can therefore never see:
+         anything below this line is invisible to a 2D laser. -->
+    <visual name="scan_band">
+      <origin xyz="0 0 0" rpy="0 0 0"/>
+      <geometry>
+        <cylinder radius="${lidar_radius*1.06}" length="0.008"/>
+      </geometry>
+      <material name="marker"/>
+    </visual>
+    <visual name="lidar_cap">
+      <origin xyz="0 0 ${lidar_height/2 + 0.004}" rpy="0 0 0"/>
+      <geometry>
+        <cylinder radius="${lidar_radius*0.8}" length="0.008"/>
+      </geometry>
+      <material name="grey"/>
     </visual>
     <collision>
@@ -192,7 +254,12 @@
   </joint>
   <link name="camera_link">
-    <visual>
-      <geometry><box size="0.02 0.06 0.02"/></geometry>
-      <material name="white"/>
+    <visual name="camera_housing">
+      <geometry><box size="0.022 0.070 0.026"/></geometry>
+      <material name="sensor"/>
+    </visual>
+    <visual name="camera_lens">
+      <origin xyz="0.013 0 0" rpy="0 ${PI/2} 0"/>
+      <geometry><cylinder radius="0.009" length="0.006"/></geometry>
+      <material name="lens"/>
     </visual>
     <collision>

Commit message: Make RViz layouts reproducible, and record two RViz rendering limits
The RViz configs looked nothing like the screenshots on a different machine.
Panel sizes are not in the readable part of an .rviz file at all: they live in
Window Geometry > QMainWindow State, a Qt-serialised blob tied to the window
size. A hand-written config without that blob makes RViz distribute panels
evenly, which is why it differed.

- scripts/bake_rviz_geometry.sh runs RViz on a 1920x1080 virtual display, sends
  Ctrl+S, and splices the saved geometry block back into the hand-written config
  so the comments are kept. All three configs now carry a layout baked at that
  resolution, and capture_rviz.sh captures at the same size, so screenshots match
  what a user sees
- both scripts now start a window manager on the virtual display; without one,
  windows cannot be focused and synthetic keystrokes never reach the application

Two rendering behaviours found while fixing this, both now documented in the
URDF and the README:

- RViz applies one material per LINK, Gazebo one per VISUAL. A link with several
  visual elements renders in RViz entirely in the first one's colour. Verified by
  reordering: moving the deck ahead of the chassis turned the whole body blue.
  The visual order is now chosen deliberately rather than by accident, and the
  chassis colour is the one RViz will actually use
- laser points reduced to 2 cm so they read as measurements on a wall rather than
  a smear over it

Also adds scripts/check_xml.py, because forbidden '--' inside XML comments has
now broken the xacro files and the world file four separate times, each time
appearing as an unhelpful "not well-formed (invalid token)".

Co-Authored-By: Claude Opus 5 <noreply@anthropic.com>

File: src/smartphone_robot/urdf/robot.urdf.xacro (robot description, xacro)
@@ -48,5 +48,5 @@
   <xacro:property name="PI" value="3.14159265359"/>
   <!-- ==================== Materials (RViz colours only) ================== -->
-  <material name="chassis">  <color rgba="0.26 0.29 0.36 1.0"/></material>
+  <material name="chassis">  <color rgba="0.34 0.40 0.50 1.0"/></material>
   <material name="deck">     <color rgba="0.20 0.58 0.86 1.0"/></material>
   <material name="tyre">     <color rgba="0.08 0.08 0.09 1.0"/></material>
@@ -76,6 +76,16 @@
   <link name="base_link">
     <!-- Several visual elements on one link. URDF allows this, and it costs nothing:
-         collision and inertia are unchanged, so physics and TF are identical. Only
-         what RViz and Gazebo draw is different. -->
+         collision and inertia are unchanged, so physics and TF are identical.
+         BUT RViz AND GAZEBO DISAGREE ABOUT MATERIALS HERE, and it is worth knowing why.
+         Gazebo renders each <visual> with its own material, so the robot appears as
+         designed: slate body, blue deck, orange bumper. RViz applies ONE material per
+         LINK  - whichever the first <visual> declares  - so in RViz the whole chassis
+         takes the 'chassis' colour and the deck and bumper are invisible. Verified by
+         reordering the visuals: putting 'deck' first turns the entire body blue.
+         So the visual order below is deliberate: 'chassis' first, because that is the
+         colour RViz will use for the whole link. The rest is detail only Gazebo shows.
+         Splitting the deck and bumper into their own links would make RViz colour them
+         too, but it would add frames to the TF tree purely for decoration, which is not
+         a trade worth making in a robot description. -->
     <visual name="chassis">
       <origin xyz="0 0 ${base_height/2}" rpy="0 0 0"/>
